Commit message: updated mechanical dimensions to match real robot

File: robot_bringup/urdf/mecanum_drive.xacro.urdf (robot description, URDF)
Before this commit: robot mecanum_vehicle, 5 links, 4 joints
Links:
- link base_link: geometry collision box size=0.52 0.42 0.1; visual box size=0.52 0.42 0.1
- link front_left_wheel: geometry collision sphere radius=0.076; visual sphere radius=0.076
- link front_right_wheel: geometry collision sphere radius=0.076; visual sphere radius=0.076
- link rear_left_wheel: geometry collision sphere radius=0.076; visual sphere radius=0.076
- link rear_right_wheel: geometry collision sphere radius=0.076; visual sphere radius=0.076
Joints:
- joint front_left_wheel_joint: origin xyz=0.6 0.5 0.3 rpy=-${pi/2} 0 0 -> xyz=0.23 0.26 0.076 rpy=-${pi/2} 0 0
- joint front_right_wheel_joint: origin xyz=0.6 -0.5 0.3 rpy=-${pi/2} 0 0 -> xyz=0.23 -0.26 0.076 rpy=-${pi/2} 0 0
- joint rear_left_wheel_joint: origin xyz=-0.6 0.5 0.3 rpy=-${pi/2} 0 0 -> xyz=-0.23 0.26 0.076 rpy=-${pi/2} 0 0
- joint rear_right_wheel_joint: origin xyz=-0.6 -0.5 0.3 rpy=-${pi/2} 0 0 -> xyz=-0.23 -0.26 0.076 rpy=-${pi/2} 0 0

Commit message: added working lidar to urdf

File: robot_bringup/urdf/mecanum_drive.xacro.urdf (robot description, URDF)
Before this commit: robot mecanum_vehicle, 5 links, 4 joints
Links:
- added link laser_frame; collision cylinder length=0.04 radius=0.05; visual cylinder length=0.04 radius=0.05
Joints:
- added joint laser_joint: type fixed, parent base_link, child laser_frame, origin xyz=0 0 0.85 rpy=0 0 0

Commit message: fixed lidar position according to real robot

File: robot_bringup/urdf/mecanum_drive.xacro.urdf (robot description, URDF)
Before this commit: robot mecanum_vehicle, 6 links, 5 joints
Joints:
- joint laser_joint: origin xyz=0 0 0.85 rpy=0 0 0 -> xyz=0 0 0.176 rpy=0 0 0

Commit message: added sim condition and minor fixes to urdf

File: robot_bringup/urdf/mecanum_drive.xacro.urdf (robot description, URDF)
Before this commit: robot mecanum_vehicle, 6 links, 5 joints
Links:
- link laser_frame: mass None -> 0.1

Commit message: Added Gazebo Sensors (#4)
* updated ak dependencies

* updated mecanum urdf

* updated mechanical dimensions to match real robot

* updated dependencies for hardware run

* moved to unstamped vel

* added josytick launch

* removed twist_mux

* added joy support and args, and updated readmes for the same

* updated readme and added stls and images

* diff push

* added working lidar to urdf

* fixed lidar position according to real robot

* added rviz config for laserscan

* changed gazebo world to add objects and change robot start pose

* fixed teleop command bug

* added sim condition and minor fixes to urdf

* minor reformatting

---------

Co-authored-by: Sarthak Mishra <sarthakminecraft@gmail.com>

File: robot_bringup/urdf/mecanum_drive.xacro.urdf (robot description, URDF)
Before this commit: robot mecanum_vehicle, 5 links, 4 joints
Links:
- added link laser_frame, mass 0.1; collision cylinder length=0.04 radius=0.05; visual cylinder length=0.04 radius=0.05
Joints:
- added joint laser_joint: type fixed, parent base_link, child laser_frame, origin xyz=0 0 0.176 rpy=0 0 0

Commit message: nav 2 working, slam working

File: robot_bringup/urdf/mecanum_drive.xacro.urdf (robot description, URDF)
Before this commit: robot mecanum_vehicle, 8 links, 7 joints
Links:
- link laser_frame: mass 0.01 -> 1

Commit message: nav 2 working, slam working

File: robot_bringup/urdf/mecanum_drive.xacro.urdf (robot description, URDF)
Before this commit: robot mecanum_vehicle, 6 links, 5 joints
Links:
- added link base_footprint
- link base_link: mass 1.5 -> 50
- link front_left_wheel: mass 2 -> 20
- link front_right_wheel: mass 2 -> 20
- link laser_frame: mass 0.1 -> 1
- link rear_left_wheel: mass 2 -> 20
- link rear_right_wheel: mass 2 -> 20
Joints:
- added joint base_footprint_joint: type fixed, parent base_link, child base_footprint, origin xyz=0.0 0.0 0.0 rpy=0 0 0

Commit message: added velodyne in urdf

File: robot_bringup/urdf/mecanum_drive.xacro.urdf (robot description, URDF)
Before this commit: robot mecanum_vehicle, 7 links, 6 joints
Links:
- added link velodyne_base_link, mass 0.83; collision cylinder length=0.0717 radius=0.0516; visual mesh filename=file://$(find robot_bringup)/meshes/VLP16/VLP16_base_1.dae
- link laser_frame: mass 1 -> 0.01; geometry visual mesh filename=file://$(find robot_bringup)/meshes/VLP16/VLP16_scan.dae
Joints:
- added joint velodyne_base_scan_joint: type fixed, parent velodyne_base_link, child laser_frame, origin xyz=0 0 0.0377 rpy=0 0 0
- joint laser_joint: child laser_frame -> velodyne_base_link

Commit message: Added Velodyne Hardware Support (#9)
* added vleodyne meshes

* added velodyne in urdf

* added velodyne dependencies

* added velodyne launch and config

File: robot_bringup/urdf/mecanum_drive.xacro.urdf (robot description, URDF)
Before this commit: robot mecanum_vehicle, 8 links, 7 joints
Links:
- link laser_frame: mass 1 -> 0.01

Commit message: added new world and related models, fixes for new lidar

File: robot_bringup/urdf/mecanum_drive.xacro.urdf (robot description, URDF)
Before this commit: robot mecanum_vehicle, 8 links, 7 joints
Joints:
- joint laser_joint: origin xyz=0 0 0.176 rpy=0 0 0 -> xyz=0.25 0 0.176 rpy=0 0 0

Commit message: ROS2 NAV2 working completely in sim (#6)
* nav 2 working, slam working

* fixed readme, added rviz config

* more changes in readme and rviz config

* added starter params for holonomic motion in nav2 config file

* updated nav2 params for holonomic mode

* Updated Front Motors to AK10-9 (#8)

* updated front motors to ak10-9

* added can command

* nav 2 working, slam working

* fixed readme, added rviz config

* more changes in readme and rviz config

* added starter params for holonomic motion in nav2 config file

* updated nav2 params for holonomic mode

* Added Velodyne Hardware Support (#9)

* added vleodyne meshes

* added velodyne in urdf

* added velodyne dependencies

* added velodyne launch and config

* removed velodyne

* added ld08 lidar driver

* removed old map files

* added new world and related models, fixes for new lidar

* addded sim map files

* nav2 holo working in sim

* added odrive usb2can commands

* moved to usb2can

* updated readme to match proper command structure

* updated maps directory and references

* removed velodyne references

* resorted maps

* updated launch file to delay nav startups

* updated readme with new params

---------

Co-authored-by: Soham Patil <sohampatil45939@gmail.com>

File: robot_bringup/urdf/mecanum_drive.xacro.urdf (robot description, URDF)
Before this commit: robot mecanum_vehicle, 6 links, 5 joints
Links:
- added link base_footprint
- added link velodyne_base_link, mass 0.83; collision cylinder length=0.0717 radius=0.0516; visual mesh filename=file://$(find robot_bringup)/meshes/VLP16/VLP16_base_1.dae
- link base_link: mass 1.5 -> 50
- link front_left_wheel: mass 2 -> 20
- link front_right_wheel: mass 2 -> 20
- link laser_frame: mass 0.1 -> 0.01; geometry visual mesh filename=file://$(find robot_bringup)/meshes/VLP16/VLP16_scan.dae
- link rear_left_wheel: mass 2 -> 20
- link rear_right_wheel: mass 2 -> 20
Joints:
- added joint base_footprint_joint: type fixed, parent base_link, child base_footprint, origin xyz=0.0 0.0 0.0 rpy=0 0 0
- added joint velodyne_base_scan_joint: type fixed, parent velodyne_base_link, child laser_frame, origin xyz=0 0 0.0377 rpy=0 0 0
- joint laser_joint: child laser_frame -> velodyne_base_link; origin xyz=0 0 0.176 rpy=0 0 0 -> xyz=0.25 0 0.176 rpy=0 0 0
